File: Glow/Plate/PCB Plate/_autosave-FR4_Bottom_Plate.kicad_pcb (KiCad board)
At the start: 2 copper layers, 139.1 x 107.7 mm, 6 parts

Commit message: Added Copper Kaguya
Parts:
- removed the G*** at (161.3, 88.8)
- added G***: LOGO, images:kaguya solder mask, F.Cu at (161.3, 87.6)
