File: Glow/Plate/PCB Plate/_autosave-FR4_Bottom_Plate.kicad_pcb (KiCad board)
At the start: 2 copper layers, 139.1 x 107.7 mm, 6 parts

Commit message: Improved silkscreen kaguya and takumi
Parts:
- removed the G*** at (161.3, 88.8)
- added G***: LOGO, images:kaguya silkscreen, F.Cu at (163.8, 88.9)
- added G***: LOGO, images:takumi silkscreen, B.Cu at (154.9, 104.1)
Other:
- board text removed: "by Nici"
