File: Glow/Plate/PCB Plate/FR4_Bottom_Plate.kicad_pcb (KiCad board)
At the start: 2 copper layers, 139.1 x 107.7 mm, 5 parts

Commit message: Moved Kaguya and Takami
Parts:
- added G***: LOGO, images:kaguya silkscreen, F.Cu at (163.8, 88.9)
- added G***: LOGO, images:takumi silkscreen, B.Cu at (154.9, 104.1)
